Commit message: Update from linux

File: linhsbot/urdf/linhsbot.xacro (robot description, xacro)
@@ -75,4 +75,14 @@
       </visual>
     </link>
+	<!--IMU-->
+	<link name="imu_link">
+      <visual>
+        <geometry>
+          <box size="0.01 0.02 0.005"/>
+        </geometry>
+        <origin rpy="0 0 0" xyz="-0.08 0 0.066"/>
+        <material name="black"/>
+      </visual>
+    </link>
     <!-- camera_link description -->
     <link name="camera_link">
@@ -141,5 +151,10 @@
       <origin xyz="0 0 0"/>
     </joint>
-	<joint name="base_to_camera_link_att" type="fixed">
+	<joint name="base_to_imu" type="fixed">
+      <parent link="base_link"/>
+      <child link="imu_link"/>
+      <origin xyz="0 0 0"/>
+    </joint>
+    <joint name="base_to_camera_link_att" type="fixed">
       <parent link="base_link"/>
       <child link="camera_link_join"/>
